Commit message: Add gripper controller support

File: src/six_dof_arm_description/urdf/six_dof_arm.urdf.xacro (robot description, xacro)
@@ -444,4 +444,15 @@
     </joint>
     <joint name="joint_6">
+      <command_interface name="position"/>
+      <state_interface name="position"/>
+      <state_interface name="velocity"/>
+    </joint>
+    <!-- gripper_ros2_control_interfaces -->
+    <joint name="gripper_left_joint">
+      <command_interface name="position"/>
+      <state_interface name="position"/>
+      <state_interface name="velocity"/>
+    </joint>
+    <joint name="gripper_right_joint">
       <command_interface name="position"/>
       <state_interface name="position"/>
